File: DIAGRAMAS/MK2560EEM-G-v1G/MK2560EM-G v1G.1.sch (EAGLE design)
At the start: 70 parts, among them U1 X-MOTOR, U2 Y-MOTOR, U3 Z-MOTOR

Commit message: pcb fixes v1G.1
- pcb bug corrections space clearance on x,y,z drivers resolution pin headers. changed for right pin headers.
- changed F5A fuse for +12v rail, for aa short cylinder standard fuse.
- pcb resized, for more space, and better alocation of components.
-
Parts:
- removed JP1, JP2, JP3, JP4, JP5, JP6, JP7, JP8: (no value), -redpic-connector:PINHD-1X3
- added SV1, SV2, SV3, SV4: (no value), con-lstb:MA03-2
- F5A: device fuse:TE5 -> special:FUSE2P
Connections:
- net +12V5A: now also F5A.1A; no longer F5A.1
- net +5V: now also SV1.2, SV1.4, SV1.6, SV2.2, SV2.4, SV2.6, SV3.2, SV3.4, SV3.6, SV4.2, SV4.4, SV4.6; no longer JP2.1, JP2.2, JP2.3, JP4.1, JP4.2, JP4.3, JP6.1, JP6.2, JP6.3, JP8.1, JP8.2, JP8.3
- net N$10: now also SV1.3; no longer JP7.2
- net N$11: now also SV1.5; no longer JP7.1
- net N$14: now also SV2.1; no longer JP1.3
- net N$15: now also SV2.3; no longer JP1.2
- net N$16: now also SV2.5; no longer JP1.1
- net N$19: now also SV3.3, U3.MS2; no longer JP3.3, U3.MS1
- net N$21: now also SV3.1, U3.MS1; no longer JP3.2, U3.MS2
- net N$22: now also SV3.5; no longer JP3.1
- net N$24: now also EXT1-MOTOR.MS2, SV4.3; no longer EXT1-MOTOR.MS3, JP5.1
- net N$25: now also EXT1-MOTOR.MS3, SV4.5; no longer EXT1-MOTOR.MS2, JP5.2
- net N$26: now also SV4.1; no longer JP5.3
- net N$27: now also F5A.2A; no longer F5A.2
- net N$9: now also SV1.1; no longer JP7.3
Other:
- note added: "MikroPrintr MK2560EM-G Rev. 1G.1 Support for RepRap Smart Controller and ESP-8266-01 Wifi Module."
- note removed: "F5A fuse is not connected on board but soldered with cables."
- note removed: "MikroPrintr MK2560EM-G Rev. 1G Support for RepRap Smart Controller and ESP-8266-01 Wifi Module."
